Commit message: Freeze Astra semantic experiment parameters

File: src/wheeltec_robot_urdf/wheeltec_robot_urdf/urdf/senior_akm_robot.urdf (robot description, URDF)
Before this commit: robot senior_akm_robot, 8 links, 7 joints
Joints:
- joint camera_joint: origin xyz=0.165778518918356 0.000945202408300414 0.089704 rpy=0 0 0 -> xyz=0.16578 0.00095 0.0474 rpy=0 -0.376226 0.002791
